File: 12vdc-supply-module.kicad_sch (KiCad schematic)
At the start: 14 parts

Commit message: Bunch more changes
Blah blah
Parts:
- removed D?: 12VDC, symbol Device:LED
- removed F?: 100A, symbol Device:Fuse
- removed J? (x2): Conn_01x01_MountingPin, symbol Connector_Generic_MountingPin:Conn_01x01_MountingPin
- removed M?: YB27VA, symbol bvm-library:5_Pin_Meter_With_Ext_Shunt
- removed R?: R_Shunt_US, symbol Device:R_Shunt_US
- removed SW_12VDC_MOD_EN_, SW_12VDC_MOD_EN_?: SW_DPDT_x2, symbol Switch:SW_DPDT_x2
- added F?: 10A, symbol Device:Fuse
- added J? (x2): Conn_01x01_MountingPin, symbol Connector_Generic_MountingPin:Conn_01x01_MountingPin
- added M?: YB27VA, symbol bvm-library:5_Pin_Meter_With_Ext_Shunt
- added SW_12VDC_POWER_EN: SW_SPST_LED_3pin, symbol bvm-library:SW_SPST_LED_3pin
Connections:
- net 12VDC_FUSED: now also F?.1, J?.1 (Pin_1), M?.3 (PWR+)
- net 12VDC_SUPPLY: now also M?.1 (+)
- net VDC_GND: now also M?.2 (-), M?.5 (COM), SW_12VDC_POWER_EN.4 (A)
- new net: J?.1 (Pin_1), M?.4 (IN+)
- new net: F?.2, SW_12VDC_POWER_EN.1
- no-connect marks 4 -> 2
Other:
- note added: "[12VDC USB POWER ACTIVE]"
- title: (none) -> Mr. Powers
- moved on the sheet: D?, F?, J?, M?, SW_12VDC_MOD_EN_A, SW_12VDC_MOD_EN_B

Commit message: Minor change across the board
I need better notes.
Parts:
- removed J? (x2): Conn_01x01_MountingPin, symbol Connector_Generic_MountingPin:Conn_01x01_MountingPin
- added D?: LED, symbol Device:LED
- added J?: Screw_Terminal_01x02, symbol Connector:Screw_Terminal_01x02
- gave numbers to parts that had none: 7
- renumbered SW_12VDC_MOD_EN_ to SW_12VDC_MOD_EN_1, SW_12VDC_POWER_EN to SW_12VDC_POWER_EN1
Connections:
- net 12VDC_FUSED: now also D?.2 (A), J?.1 (Pin_1)
- net 12VDC_SUPPLY: now also SW_12VDC_POWER_EN1.2
- net VDC_GND: now also SW_12VDC_POWER_EN1.3 (A), D?.1 (K); no longer SW_12VDC_POWER_EN1.4 (A)
- net at M4.4 (IN+): now also J?.2 (Pin_2)
- no-connect marks 2 -> 4
Changed lines of the file:
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@@
   (junction (at 187.96 57.15) (diameter 0) (color 255 255 0 1)
+  )
+  (junction (at 114.3 110.49) (diameter 0) (color 0 0 0 0)
   )
   (junction (at 114.3 124.46) (diameter 0) (color 0 0 0 0)
@@
   (no_connect (at 168.91 53.34))
   (no_connect (at 170.18 67.31))
+  (no_connect (at 90.17 69.85))
+  (no_connect (at 90.17 53.34))
   (wire (pts (xy 187.96 57.15) (xy 187.96 64.77))
     (stroke (width 0) (type default) (color 255 255 0 1))
@@
     (stroke (width 0) (type default) (color 255 255 0 1))
   )
+  (wire (pts (xy 114.3 95.25) (xy 182.88 95.25))
+    (stroke (width 0) (type default) (color 0 0 0 0))
+  )
   (wire (pts (xy 187.96 64.77) (xy 180.34 64.77))
     (stroke (width 0) (type default) (color 255 255 0 1))
   )
+  (wire (pts (xy 114.3 95.25) (xy 114.3 110.49))
+    (stroke (width 0) (type default) (color 0 0 0 0))
+  )
   (wire (pts (xy 95.25 48.26) (xy 119.38 48.26))
     (stroke (width 0) (type default) (color 0 0 0 0))
@@
     (stroke (width 0) (type default) (color 0 0 0 0))
   )
+  (wire (pts (xy 129.54 132.08) (xy 130.81 132.08))
+    (stroke (width 0) (type default) (color 0 0 0 0))
+  )
   (wire (pts (xy 119.38 62.23) (xy 119.38 48.26))
     (stroke (width 0) (type default) (color 0 0 0 0))
@@
   (wire (pts (xy 168.91 124.46) (xy 189.23 124.46))
     (stroke (width 0) (type default) (color 255 255 0 1))
+  )
+  (wire (pts (xy 181.61 110.49) (xy 189.23 110.49))
+    (stroke (width 0) (type default) (color 0 0 0 0))
   )
   (wire (pts (xy 185.42 72.39) (xy 153.67 72.39))
@@
     )
   )
+  (global_label "VDC_GND" (shape input) (at 190.5 95.25 0) (fields_autoplaced)
+    (effects (font (size 1.27 1.27)) (justify left))
+    (property "Intersheet References" "${INTERSHEET_REFS}" (id 0) (at 201.3798 95.1706 0)
+      (effects (font (size 1.27 1.27)) (justify left))
+    )
+  )
   (global_label "VDC_GND" (shape input) (at 185.42 72.39 0) (fields_autoplaced)
     (effects (font (size 1.27 1.27)) (justify left))
@@
     )
   )
-  (global_label "VDC_GND" (shape input) (at 130.81 132.08 180) (fields_autoplaced)
+  (global_label "VDC_GND" (shape input) (at 129.54 132.08 180) (fields_autoplaced)
     (effects (font (size 1.27 1.27)) (justify right))
-    (property "Intersheet References" "${INTERSHEET_REFS}" (id 0) (at 119.9302 132.0006 0)
+    (property "Intersheet References" "${INTERSHEET_REFS}" (id 0) (at 118.6602 132.0006 0)
       (effects (font (size 1.27 1.27)) (justify right))
     )
@@
   (symbol (lib_id "Switch:SW_DPDT_x2") (at 173.99 50.8 0) (mirror y) (unit 1)
     (in_bom yes) (on_board yes) (fields_autoplaced)
-    (property "Reference" "SW_12VDC_MOD_EN_" (id 0) (at 173.99 43.18 0))
+    (property "Reference" "SW_12VDC_MOD_EN_1" (id 0) (at 173.99 43.18 0))
     (property "Value" "SW_DPDT_x2" (id 1) (at 173.99 45.72 0))
     (property "Footprint" "" (id 2) (at 173.99 50.8 0)
@@
   (symbol (lib_id "bvm-library:5_Pin_Meter_With_Ext_Shunt") (at 138.43 129.54 0) (unit 1)
     (in_bom yes) (on_board yes) (fields_autoplaced)
-    (property "Reference" "M?" (id 0) (at 143.51 114.3 0))
+    (property "Reference" "M4" (id 0) (at 143.51 114.3 0))
     (property "Value" "YB27VA" (id 1) (at 143.51 116.84 0))
     (property "Footprint" "" (id 2) (at 138.43 129.54 0)
@@
     (pin "5")
   )
-  (symbol (lib_id "Connector_Generic_MountingPin:Conn_01x01_MountingPin") (at 82.55 127 0) (mirror y) (unit 1)
+  (symbol (lib_id "Device:LED") (at 186.69 95.25 0) (mirror y) (unit 1)
     (in_bom yes) (on_board yes) (fields_autoplaced)
-    (property "Reference" "J?" (id 0) (at 80.01 127.3555 0)
-      (effects (font (size 1.27 1.27)) (justify left))
-    )
-    (property "Value" "Conn_01x01_MountingPin" (id 1) (at 80.01 128.6255 0)
-      (effects (font (size 1.27 1.27)) (justify left) hide)
-    )
-    (property "Footprint" "" (id 2) (at 82.55 127 0)
+    (property "Reference" "D?" (id 0) (at 188.2775 88.9 0))
+    (property "Value" "LED" (id 1) (at 188.2775 91.44 0))
+    (property "Footprint" "" (id 2) (at 186.69 95.25 0)
       (effects (font (size 1.27 1.27)) hide)
     )
-    (property "Datasheet" "~" (id 3) (at 82.55 127 0)
+    (property "Datasheet" "~" (id 3) (at 186.69 95.25 0)
       (effects (font (size 1.27 1.27)) hide)
     )
     (pin "1")
-    (pin "MP")
+    (pin "2")
+  )
+  (symbol (lib_id "Connector:Screw_Terminal_01x02") (at 82.55 124.46 0) (mirror y) (unit 1)
+    (in_bom yes) (on_board yes) (fields_autoplaced)
+    (property "Reference" "J?" (id 0) (at 82.55 120.65 0))
+    (property "Value" "Screw_Terminal_01x02" (id 1) (at 82.55 120.65 0)
+      (effects (font (size 1.27 1.27)) hide)
+    )
+    (property "Footprint" "" (id 2) (at 82.55 124.46 0)
+      (effects (font (size 1.27 1.27)) hide)
+    )
+    (property "Datasheet" "~" (id 3) (at 82.55 124.46 0)
+      (effects (font (size 1.27 1.27)) hide)
+    )
+    (pin "1")
+    (pin "2")
   )
   (symbol (lib_id "Device:LED") (at 162.56 62.23 0) (unit 1)
     (in_bom yes) (on_board yes)
-    (property "Reference" "D?" (id 0) (at 162.56 68.58 0))
+    (property "Reference" "D2" (id 0) (at 162.56 68.58 0))
     (property "Value" "12VDC" (id 1) (at 161.29 66.04 0))
     (property "Footprint" "" (id 2) (at 162.56 62.23 0)
@@
   (symbol (lib_id "bvm-library:5_Pin_Meter_With_Ext_Shunt") (at 135.89 67.31 0) (unit 1)
     (in_bom yes) (on_board yes) (fields_autoplaced)
-    (property "Reference" "M?" (id 0) (at 140.97 52.07 0))
+    (property "Reference" "M3" (id 0) (at 140.97 52.07 0))
     (property "Value" "YB27VA" (id 1) (at 140.97 54.61 0))
     (property "Footprint" "" (id 2) (at 135.89 67.31 0)
@@
     (pin "5")
   )
-  (symbol (lib_id "Connector_Generic_MountingPin:Conn_01x01_MountingPin") (at 82.55 124.46 180) (unit 1)
-    (in_bom yes) (on_board yes) (fields_autoplaced)
-    (property "Reference" "J?" (id 0) (at 80.01 124.1043 0)
-      (effects (font (size 1.27 1.27)) (justify left))
-    )
-    (property "Value" "Conn_01x01_MountingPin" (id 1) (at 80.01 122.8345 0)
-      (effects (font (size 1.27 1.27)) (justify left) hide)
-    )
-    (property "Footprint" "" (id 2) (at 82.55 124.46 0)
-      (effects (font (size 1.27 1.27)) hide)
-    )
-    (property "Datasheet" "~" (id 3) (at 82.55 124.46 0)
-      (effects (font (size 1.27 1.27)) hide)
-    )
-    (pin "1")
-    (pin "MP")
-  )
   (symbol (lib_id "Switch:SW_DPDT_x2") (at 175.26 64.77 0) (mirror y) (unit 2)
     (in_bom yes) (on_board yes) (fields_autoplaced)
-    (property "Reference" "SW_12VDC_MOD_EN_" (id 0) (at 175.26 57.15 0))
+    (property "Reference" "SW_12VDC_MOD_EN_1" (id 0) (at 175.26 57.15 0))
     (property "Value" "SW_DPDT_x2" (id 1) (at 175.26 59.69 0))
     (property "Footprint" "" (id 2) (at 175.26 64.77 0)
@@
   (symbol (lib_id "Device:Fuse") (at 152.4 48.26 90) (unit 1)
     (in_bom yes) (on_board yes) (fields_autoplaced)
-    (property "Reference" "F?" (id 0) (at 152.4 41.91 90))
+    (property "Reference" "F3" (id 0) (at 152.4 41.91 90))
     (property "Value" "10A" (id 1) (at 152.4 44.45 90))
     (property "Footprint" "" (id 2) (at 152.4 50.038 90)
@@
   (symbol (lib_id "Connector_Generic_MountingPin:Conn_01x01_MountingPin") (at 90.17 64.77 0) (mirror y) (unit 1)
     (in_bom yes) (on_board yes) (fields_autoplaced)
-    (property "Reference" "J?" (id 0) (at 90.17 60.96 0))
+    (property "Reference" "J6" (id 0) (at 90.17 60.96 0))
     (property "Value" "Conn_01x01_MountingPin" (id 1) (at 87.63 66.3955 0)
       (effects (font (size 1.27 1.27)) (justify left) hide)
@@
   (symbol (lib_id "Device:Fuse") (at 143.51 110.49 90) (unit 1)
     (in_bom yes) (on_board yes) (fields_autoplaced)
-    (property "Reference" "F?" (id 0) (at 143.51 104.14 90))
+    (property "Reference" "F2" (id 0) (at 143.51 104.14 90))
     (property "Value" "10A" (id 1) (at 143.51 106.68 90))
     (property "Footprint" "" (id 2) (at 143.51 112.268 90)
@@
   (symbol (lib_id "Connector_Generic_MountingPin:Conn_01x01_MountingPin") (at 90.17 48.26 0) (mirror y) (unit 1)
     (in_bom yes) (on_board yes) (fields_autoplaced)
-    (property "Reference" "J?" (id 0) (at 90.17 44.45 0))
+    (property "Reference" "J5" (id 0) (at 90.17 44.45 0))
     (property "Value" "Conn_01x01_MountingPin" (id 1) (at 87.63 49.8855 0)
       (effects (font (size 1.27 1.27)) (justify left) hide)
@@
   (symbol (lib_id "bvm-library:SW_SPST_LED_3pin") (at 176.53 113.03 0) (unit 1)
     (in_bom yes) (on_board yes) (fields_autoplaced)
-    (property "Reference" "SW_12VDC_POWER_EN" (id 0) (at 175.895 104.14 0))
+    (property "Reference" "SW_12VDC_POWER_EN1" (id 0) (at 175.895 104.14 0))
     (property "Value" "SW_SPST_LED_3pin" (id 1) (at 175.895 106.68 0))
     (property "Footprint" "" (id 2) (at 176.53 105.41 0)
@@
     (pin "1")
     (pin "2")
-    (pin "4")
+    (pin "3")
   )
 )
