File: variable-vdc-supply-module.kicad_sch (KiCad schematic)
At the start: 0 parts

Commit message: Bunch more changes
Blah blah
Other:
- title: (none) -> Mr. Powers
Changed lines of the file:
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@@
   (paper "A4")
   (title_block
+    (title "Mr. Powers")
     (date "2022-05-20")
     (rev "0.0.0-draft")
