File: 12vdc-ext-supply-module.kicad_sch (KiCad schematic)
At the start: 5 parts

Commit message: Minor change across the board
I need better notes.
Parts:
- gave numbers to parts that had none: 3
- renumbered F_12VDC_EXT_SUPPLY to F_12VDC_EXT_SUPPLY1, SW_12VDC_EXT_SUPPLY to SW_12VDC_EXT_SUPPLY1
Connections:
- net VDC_GND: now also SW_12VDC_EXT_SUPPLY1.3 (A); no longer SW_12VDC_EXT_SUPPLY1.4 (A)
Changed lines of the file:
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@@
   (symbol (lib_id "Connector:Conn_01x02_Male") (at 80.01 72.39 0) (unit 1)
     (in_bom yes) (on_board yes) (fields_autoplaced)
-    (property "Reference" "J?" (id 0) (at 80.645 67.31 0))
+    (property "Reference" "J22" (id 0) (at 80.645 67.31 0))
     (property "Value" "XT60" (id 1) (at 80.645 69.85 0))
     (property "Footprint" "" (id 2) (at 80.01 72.39 0)
@@
   (symbol (lib_id "Device:LED") (at 118.11 69.85 0) (unit 1)
     (in_bom yes) (on_board yes) (fields_autoplaced)
-    (property "Reference" "D?" (id 0) (at 116.5225 63.5 0))
+    (property "Reference" "D12" (id 0) (at 116.5225 63.5 0))
     (property "Value" "12VDC RED" (id 1) (at 116.5225 66.04 0))
     (property "Footprint" "" (id 2) (at 118.11 69.85 0)
@@
   (symbol (lib_id "bvm-library:SW_SPST_LED_3pin") (at 166.37 72.39 0) (mirror y) (unit 1)
     (in_bom yes) (on_board yes) (fields_autoplaced)
-    (property "Reference" "SW_12VDC_EXT_SUPPLY" (id 0) (at 167.005 63.5 0))
+    (property "Reference" "SW_12VDC_EXT_SUPPLY1" (id 0) (at 167.005 63.5 0))
     (property "Value" "SW_SPST_LED_3pin" (id 1) (at 167.005 66.04 0))
     (property "Footprint" "" (id 2) (at 166.37 64.77 0)
@@
     (pin "1")
     (pin "2")
-    (pin "4")
+    (pin "3")
   )
   (symbol (lib_id "Device:LED") (at 137.16 73.66 90) (unit 1)
     (in_bom yes) (on_board yes) (fields_autoplaced)
-    (property "Reference" "D?" (id 0) (at 140.97 73.9774 90)
+    (property "Reference" "D13" (id 0) (at 140.97 73.9774 90)
       (effects (font (size 1.27 1.27)) (justify right))
     )
@@
   (symbol (lib_id "Device:Fuse") (at 140.97 69.85 270) (unit 1)
     (in_bom yes) (on_board yes) (fields_autoplaced)
-    (property "Reference" "F_12VDC_EXT_SUPPLY" (id 0) (at 140.97 63.5 90))
+    (property "Reference" "F_12VDC_EXT_SUPPLY1" (id 0) (at 140.97 63.5 90))
     (property "Value" "10A" (id 1) (at 140.97 66.04 90))
     (property "Footprint" "" (id 2) (at 140.97 68.072 90)
