File: 5vdc-supply-module.kicad_sch (KiCad schematic)
At the start: 0 parts

Commit message: Draft 5VDC Supply Schematic
Parts:
- added F? (x2): Fuse, symbol Device:Fuse
- added J? (x4): Conn_01x01_MountingPin, symbol Connector_Generic_MountingPin:Conn_01x01_MountingPin
- added M? (x2): YB27VA, symbol bvm-library:5_Pin_Meter_With_Ext_Shunt
- added R?: R_Shunt_US, symbol Device:R_Shunt_US
- added SW_SYSPOWER? (x2): SW_SPST_LED, symbol Switch:SW_SPST_LED
Connections:
- new net: M?.1 (VDC), SW_SYSPOWER?.2, SW_SYSPOWER?.4 (A) (x2)
- new net: M?.4 (Shunt-), R?.2
- new net: M?.5 (GND), R?.3
- new net: J?.1 (Pin_1), R?.1
- new net: J?.1 (Pin_1), M?.4 (Shunt-)
- new net 12VDC_SUPPLY: SW_SYSPOWER?.1, SW_SYSPOWER?.1
- new net 5VDC_FUSED: F?.1, F?.1, J?.1 (Pin_1), J?.1 (Pin_1), M?.3 (Shunt+), M?.3 (Shunt+)
- new net 5VDC_SUPPLY: F?.2, F?.2
- new net VDC_GND: M?.2 (GND), M?.2 (GND), M?.5 (GND), R?.4, SW_SYSPOWER?.3 (K), SW_SYSPOWER?.3 (K)
Other:
- note added: "5VDC TERM"
- note added: "< 10Amp Version"
- note added: "> 10Amp Version"
- note added: "Can I make use of some kind of switch that would allow me to enable/disable the shunt?"
- note added: "VDC GND TERM"
- note added: "VDC_IN"
- note added: "VDC_LOAD"

Commit message: Save more changes
Started Fan Control
Created VDC Meter Template
Fleshed out 12, 5, 5-usb, and 3.3 modules
Parts:
- added D?: 12VDC, symbol Device:LED
- added F?: 10A, symbol Device:Fuse
- added J? (x2): Conn_01x01_MountingPin, symbol Connector_Generic_MountingPin:Conn_01x01_MountingPin
- added M?: YB27VA, symbol bvm-library:5_Pin_Meter_With_Ext_Shunt
- added SW_5VDC_MOD_EN_: SW_DPDT_x2, symbol Switch:SW_DPDT_x2
Connections:
- net 12VDC_SUPPLY: now also SW_5VDC_MOD_EN_.5 (B)
- net 5VDC_FUSED: now also F?.1, J?.1 (Pin_1), M?.3 (PWR+)
- net 5VDC_SUPPLY: now also SW_5VDC_MOD_EN_.2 (B)
- net VDC_GND: now also M?.2 (-), M?.5 (COM)
- new net: J?.1 (Pin_1), M?.4 (IN+)
- new net: D?.1 (K), M?.1 (+)
- new net: D?.2 (A), SW_5VDC_MOD_EN_.4 (A)
- new net: F?.2, SW_5VDC_MOD_EN_.1 (A)
- no-connect marks 0 -> 2
Other:
- note added: "<=10A"
- moved on the sheet: F?, J?, M?, R?, SW_SYSPOWER?

Commit message: Bunch more changes
Blah blah
Parts:
- removed F? (x2): Fuse, symbol Device:Fuse
- removed J? (x4): Conn_01x01_MountingPin, symbol Connector_Generic_MountingPin:Conn_01x01_MountingPin
- removed M? (x2): YB27VA, symbol bvm-library:5_Pin_Meter_With_Ext_Shunt
- removed R?: R_Shunt_US, symbol Device:R_Shunt_US
- removed SW_SYSPOWER? (x2): SW_SPST_LED, symbol Switch:SW_SPST_LED
Other:
- note removed: "5VDC TERM"
- note removed: "< 10Amp Version"
- note removed: "> 10Amp Version"
- note removed: "Can I make use of some kind of switch that would allow me to enable/disable the shunt?"
- note removed: "VDC GND TERM"
- note removed: "VDC_IN"
- note removed: "VDC_LOAD"
- title: (none) -> Mr. Powers

Commit message: Minor change across the board
I need better notes.
Parts:
- gave numbers to parts that had none: 5
- renumbered SW_5VDC_MOD_EN_ to SW_5VDC_MOD_EN_1
Changed lines of the file:
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@@
   (symbol (lib_id "Connector_Generic_MountingPin:Conn_01x01_MountingPin") (at 119.38 36.83 0) (mirror y) (unit 1)
     (in_bom yes) (on_board yes) (fields_autoplaced)
-    (property "Reference" "J?" (id 0) (at 119.38 33.02 0))
+    (property "Reference" "J1" (id 0) (at 119.38 33.02 0))
     (property "Value" "Conn_01x01_MountingPin" (id 1) (at 116.84 38.4555 0)
       (effects (font (size 1.27 1.27)) (justify left) hide)
@@
   (symbol (lib_id "Connector_Generic_MountingPin:Conn_01x01_MountingPin") (at 119.38 53.34 0) (mirror y) (unit 1)
     (in_bom yes) (on_board yes) (fields_autoplaced)
-    (property "Reference" "J?" (id 0) (at 119.38 49.53 0))
+    (property "Reference" "J2" (id 0) (at 119.38 49.53 0))
     (property "Value" "Conn_01x01_MountingPin" (id 1) (at 116.84 54.9655 0)
       (effects (font (size 1.27 1.27)) (justify left) hide)
@@
   (symbol (lib_id "Device:LED") (at 191.77 50.8 0) (unit 1)
     (in_bom yes) (on_board yes)
-    (property "Reference" "D?" (id 0) (at 191.77 57.15 0))
+    (property "Reference" "D1" (id 0) (at 191.77 57.15 0))
     (property "Value" "12VDC" (id 1) (at 190.5 54.61 0))
     (property "Footprint" "" (id 2) (at 191.77 50.8 0)
@@
   (symbol (lib_id "Device:Fuse") (at 181.61 36.83 90) (unit 1)
     (in_bom yes) (on_board yes) (fields_autoplaced)
-    (property "Reference" "F?" (id 0) (at 181.61 30.48 90))
+    (property "Reference" "F1" (id 0) (at 181.61 30.48 90))
     (property "Value" "10A" (id 1) (at 181.61 33.02 90))
     (property "Footprint" "" (id 2) (at 181.61 38.608 90)
@@
   (symbol (lib_id "bvm-library:5_Pin_Meter_With_Ext_Shunt") (at 165.1 55.88 0) (unit 1)
     (in_bom yes) (on_board yes) (fields_autoplaced)
-    (property "Reference" "M?" (id 0) (at 170.18 40.64 0))
+    (property "Reference" "M2" (id 0) (at 170.18 40.64 0))
     (property "Value" "YB27VA" (id 1) (at 170.18 43.18 0))
     (property "Footprint" "" (id 2) (at 165.1 55.88 0)
@@
   (symbol (lib_id "Switch:SW_DPDT_x2") (at 204.47 53.34 0) (mirror y) (unit 2)
     (in_bom yes) (on_board yes) (fields_autoplaced)
-    (property "Reference" "SW_5VDC_MOD_EN_" (id 0) (at 204.47 45.72 0))
+    (property "Reference" "SW_5VDC_MOD_EN_1" (id 0) (at 204.47 45.72 0))
     (property "Value" "SW_DPDT_x2" (id 1) (at 204.47 48.26 0))
     (property "Footprint" "" (id 2) (at 204.47 53.34 0)
@@
   (symbol (lib_id "Switch:SW_DPDT_x2") (at 203.2 39.37 0) (mirror y) (unit 1)
     (in_bom yes) (on_board yes) (fields_autoplaced)
-    (property "Reference" "SW_5VDC_MOD_EN_" (id 0) (at 203.2 31.75 0))
+    (property "Reference" "SW_5VDC_MOD_EN_1" (id 0) (at 203.2 31.75 0))
     (property "Value" "SW_DPDT_x2" (id 1) (at 203.2 34.29 0))
     (property "Footprint" "" (id 2) (at 203.2 39.37 0)
