File: always-on-usb.kicad_sch (KiCad schematic)
At the start: 3 parts

Commit message: Minor change across the board
I need better notes.
Parts:
- gave numbers to parts that had none: 3
Changed lines of the file:
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@@
   (symbol (lib_id "Device:LED") (at 160.02 54.61 270) (mirror x) (unit 1)
     (in_bom yes) (on_board yes) (fields_autoplaced)
-    (property "Reference" "D?" (id 0) (at 162.56 54.9274 90)
+    (property "Reference" "D11" (id 0) (at 162.56 54.9274 90)
       (effects (font (size 1.27 1.27)) (justify left))
     )
@@
   (symbol (lib_id "Device:LED") (at 146.05 86.36 0) (unit 1)
     (in_bom yes) (on_board yes) (fields_autoplaced)
-    (property "Reference" "D?" (id 0) (at 144.4625 80.01 0))
+    (property "Reference" "D9" (id 0) (at 144.4625 80.01 0))
     (property "Value" "5VDC GREEN" (id 1) (at 144.4625 82.55 0))
     (property "Footprint" "" (id 2) (at 146.05 86.36 0)
@@
   (symbol (lib_id "bvm-library:USB_PWR_A") (at 106.68 86.36 0) (unit 1)
     (in_bom no) (on_board no) (fields_autoplaced)
-    (property "Reference" "J?" (id 0) (at 106.68 73.66 0))
+    (property "Reference" "#J020" (id 0) (at 106.68 73.66 0))
     (property "Value" "USB_PWR_A" (id 1) (at 106.68 76.2 0))
     (property "Footprint" "" (id 2) (at 110.49 87.63 0)
@@
   (symbol (lib_id "bvm-library:USB_PWR_A") (at 106.68 113.03 0) (unit 1)
     (in_bom no) (on_board no) (fields_autoplaced)
-    (property "Reference" "J?" (id 0) (at 106.68 100.33 0))
+    (property "Reference" "#J021" (id 0) (at 106.68 100.33 0))
     (property "Value" "USB_PWR_A" (id 1) (at 106.68 102.87 0))
     (property "Footprint" "" (id 2) (at 110.49 114.3 0)
@@
   (symbol (lib_id "Device:LED") (at 146.05 113.03 0) (unit 1)
     (in_bom yes) (on_board yes) (fields_autoplaced)
-    (property "Reference" "D?" (id 0) (at 144.4625 106.68 0))
+    (property "Reference" "D10" (id 0) (at 144.4625 106.68 0))
     (property "Value" "5VDC GREEN" (id 1) (at 144.4625 109.22 0))
     (property "Footprint" "" (id 2) (at 146.05 113.03 0)
