File: fan-control-module.kicad_sch (KiCad schematic)
At the start: 1 part

Commit message: Bunch more changes
Blah blah
Parts:
- removed U?: 12VDC_PWM_FAN_DRIVER, symbol bvm-library:12VDC_PWM_FAN_DRIVER
- added U?: 12VDC_PWM_FAN_DRIVER, symbol bvm-library:12VDC_PWM_FAN_DRIVER
Connections:
- new net 12VDC_SUPPLY: U?. (12VDC-)
- new net VDC_GND: U?. (12VDC-)
- no-connect marks 0 -> 12

Commit message: Minor change across the board
I need better notes.
Parts:
- gave numbers to parts that had none: 1
Changed lines of the file:
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@@
   (symbol (lib_id "bvm-library:12VDC_PWM_FAN_DRIVER") (at 115.57 124.46 0) (mirror y) (unit 1)
     (in_bom yes) (on_board yes)
-    (property "Reference" "U?" (id 0) (at 115.57 116.84 0))
+    (property "Reference" "U3" (id 0) (at 115.57 116.84 0))
     (property "Value" "12VDC_PWM_FAN_DRIVER" (id 1) (at 115.57 121.92 0))
     (property "Footprint" "" (id 2) (at 115.57 124.46 0)
