File: vdc-meter-module.kicad_sch (KiCad schematic)
At the start: 0 parts

Commit message: Draft 5VDC Supply Schematic
Parts:
- added J? (x4): Conn_01x01_MountingPin, symbol Connector_Generic_MountingPin:Conn_01x01_MountingPin
- added M?: 5_Pin_Meter_With_Ext_Shunt, symbol bvm-library:5_Pin_Meter_With_Ext_Shunt
- added R?: R_Shunt_US, symbol Device:R_Shunt_US
- added SW_SYSPOWER?: SW_SPST_LED, symbol Switch:SW_SPST_LED
Connections:
- new net: J?.1 (Pin_1), M?.1 (VDC), R?.1, SW_SYSPOWER?.2, SW_SYSPOWER?.4 (A)
- new net: M?.3 (Shunt+), R?.2
- new net: M?.4 (Shunt-), R?.3
- new net: J?.1 (Pin_1), R?.4
- new net 12VDC_SUPPLY: SW_SYSPOWER?.1
- new net VDC_GND: J?.1 (Pin_1), J?.1 (Pin_1), M?.2 (GND), M?.5 (GND), SW_SYSPOWER?.3 (K)
Changed lines of the file:
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@@
     (company "eatmellc")
   )
+  (junction (at 179.07 74.93) (diameter 0) (color 0 0 0 0)
+  )
+  (junction (at 60.96 96.52) (diameter 0) (color 0 0 0 0)
+  )
+  (junction (at 60.96 30.48) (diameter 0) (color 0 0 0 0)
+  )
+  (junction (at 152.4 66.04) (diameter 0) (color 0 0 0 0)
+  )
+  (junction (at 78.74 40.64) (diameter 0) (color 0 0 0 0)
+  )
+  (junction (at 144.78 66.04) (diameter 0) (color 0 0 0 0)
+  )
+  (junction (at 179.07 68.58) (diameter 0) (color 0 0 0 0)
+  )
+  (wire (pts (xy 144.78 40.64) (xy 144.78 66.04))
+    (stroke (width 0) (type default) (color 0 0 0 0))
+  )
+  (wire (pts (xy 179.07 74.93) (xy 137.16 74.93))
+    (stroke (width 0) (type default) (color 0 0 0 0))
+  )
+  (wire (pts (xy 22.86 25.4) (xy 22.86 104.14))
+    (stroke (width 0) (type default) (color 0 0 0 0))
+  )
+  (wire (pts (xy 60.96 30.48) (xy 60.96 25.4))
+    (stroke (width 0) (type default) (color 0 0 0 0))
+  )
+  (wire (pts (xy 214.63 30.48) (xy 214.63 74.93))
+    (stroke (width 0) (type default) (color 0 0 0 0))
+  )
+  (wire (pts (xy 78.74 71.12) (xy 78.74 86.36))
+    (stroke (width 0) (type default) (color 0 0 0 0))
+  )
+  (wire (pts (xy 78.74 40.64) (xy 144.78 40.64))
+    (stroke (width 0) (type default) (color 0 0 0 0))
+  )
+  (wire (pts (xy 60.96 30.48) (xy 214.63 30.48))
+    (stroke (width 0) (type default) (color 0 0 0 0))
+  )
+  (wire (pts (xy 111.76 96.52) (xy 60.96 96.52))
+    (stroke (width 0) (type default) (color 0 0 0 0))
+  )
+  (wire (pts (xy 157.48 66.04) (xy 152.4 66.04))
+    (stroke (width 0) (type default) (color 0 0 0 0))
+  )
+  (wire (pts (xy 144.78 66.04) (xy 137.16 66.04))
+    (stroke (width 0) (type default) (color 0 0 0 0))
+  )
+  (wire (pts (xy 111.76 63.5) (xy 111.76 66.04))
+    (stroke (width 0) (type default) (color 0 0 0 0))
+  )
+  (wire (pts (xy 167.64 68.58) (xy 179.07 68.58))
+    (stroke (width 0) (type default) (color 0 0 0 0))
+  )
+  (wire (pts (xy 167.64 66.04) (xy 182.88 66.04))
+    (stroke (width 0) (type default) (color 0 0 0 0))
+  )
+  (wire (pts (xy 60.96 40.64) (xy 78.74 40.64))
+    (stroke (width 0) (type default) (color 0 0 0 0))
+  )
+  (wire (pts (xy 78.74 86.36) (xy 60.96 86.36))
+    (stroke (width 0) (type default) (color 0 0 0 0))
+  )
+  (wire (pts (xy 152.4 66.04) (xy 144.78 66.04))
+    (stroke (width 0) (type default) (color 0 0 0 0))
+  )
+  (wire (pts (xy 82.55 68.58) (xy 111.76 68.58))
+    (stroke (width 0) (type default) (color 0 0 0 0))
+  )
+  (wire (pts (xy 179.07 68.58) (xy 182.88 68.58))
+    (stroke (width 0) (type default) (color 0 0 0 0))
+  )
+  (wire (pts (xy 152.4 66.04) (xy 152.4 68.58))
+    (stroke (width 0) (type default) (color 0 0 0 0))
+  )
+  (wire (pts (xy 152.4 68.58) (xy 157.48 68.58))
+    (stroke (width 0) (type default) (color 0 0 0 0))
+  )
+  (wire (pts (xy 60.96 25.4) (xy 22.86 25.4))
+    (stroke (width 0) (type default) (color 0 0 0 0))
+  )
+  (wire (pts (xy 82.55 63.5) (xy 111.76 63.5))
+    (stroke (width 0) (type default) (color 0 0 0 0))
+  )
+  (wire (pts (xy 137.16 71.12) (xy 137.16 74.93))
+    (stroke (width 0) (type default) (color 0 0 0 0))
+  )
+  (wire (pts (xy 111.76 73.66) (xy 111.76 96.52))
+    (stroke (width 0) (type default) (color 0 0 0 0))
+  )
+  (wire (pts (xy 78.74 40.64) (xy 78.74 60.96))
+    (stroke (width 0) (type default) (color 0 0 0 0))
+  )
+  (wire (pts (xy 179.07 68.58) (xy 179.07 74.93))
+    (stroke (width 0) (type default) (color 0 0 0 0))
+  )
+  (wire (pts (xy 22.86 104.14) (xy 60.96 104.14))
+    (stroke (width 0) (type default) (color 0 0 0 0))
+  )
+  (wire (pts (xy 214.63 74.93) (xy 179.07 74.93))
+    (stroke (width 0) (type default) (color 0 0 0 0))
+  )
+  (wire (pts (xy 60.96 104.14) (xy 60.96 96.52))
+    (stroke (width 0) (type default) (color 0 0 0 0))
+  )
+  (global_label "VDC_GND" (shape input) (at 182.88 68.58 0) (fields_autoplaced)
+    (effects (font (size 1.27 1.27)) (justify left))
+    (property "Intersheet References" "${INTERSHEET_REFS}" (id 0) (at 193.7598 68.5006 0)
+      (effects (font (size 1.27 1.27)) (justify left))
+    )
+  )
+  (global_label "12VDC_SUPPLY" (shape input) (at 182.88 66.04 0) (fields_autoplaced)
+    (effects (font (size 1.27 1.27)) (justify left))
+    (property "Intersheet References" "${INTERSHEET_REFS}" (id 0) (at 199.505 65.9606 0)
+      (effects (font (size 1.27 1.27)) (justify left))
+    )
+  )
+  (symbol (lib_id "Connector_Generic_MountingPin:Conn_01x01_MountingPin") (at 55.88 30.48 0) (mirror y) (unit 1)
+    (in_bom yes) (on_board yes) (fields_autoplaced)
+    (property "Reference" "J?" (id 0) (at 53.34 29.5655 0)
+      (effects (font (size 1.27 1.27)) (justify left))
+    )
+    (property "Value" "Conn_01x01_MountingPin" (id 1) (at 53.34 32.1055 0)
+      (effects (font (size 1.27 1.27)) (justify left))
+    )
+    (property "Footprint" "" (id 2) (at 55.88 30.48 0)
+      (effects (font (size 1.27 1.27)) hide)
+    )
+    (property "Datasheet" "~" (id 3) (at 55.88 30.48 0)
+      (effects (font (size 1.27 1.27)) hide)
+    )
+    (pin "1")
+    (pin "MP")
+  )
+  (symbol (lib_id "Connector_Generic_MountingPin:Conn_01x01_MountingPin") (at 55.88 96.52 0) (mirror y) (unit 1)
+    (in_bom yes) (on_board yes) (fields_autoplaced)
+    (property "Reference" "J?" (id 0) (at 53.34 95.6055 0)
+      (effects (font (size 1.27 1.27)) (justify left))
+    )
+    (property "Value" "Conn_01x01_MountingPin" (id 1) (at 53.34 98.1455 0)
+      (effects (font (size 1.27 1.27)) (justify left))
+    )
+    (property "Footprint" "" (id 2) (at 55.88 96.52 0)
+      (effects (font (size 1.27 1.27)) hide)
+    )
+    (property "Datasheet" "~" (id 3) (at 55.88 96.52 0)
+      (effects (font (size 1.27 1.27)) hide)
+    )
+    (pin "1")
+    (pin "MP")
+  )
+  (symbol (lib_id "Switch:SW_SPST_LED") (at 162.56 68.58 0) (mirror y) (unit 1)
+    (in_bom yes) (on_board yes) (fields_autoplaced)
+    (property "Reference" "SW_SYSPOWER?" (id 0) (at 163.195 59.69 0))
+    (property "Value" "SW_SPST_LED" (id 1) (at 163.195 62.23 0))
+    (property "Footprint" "" (id 2) (at 162.56 60.96 0)
+      (effects (font (size 1.27 1.27)) hide)
+    )
+    (property "Datasheet" "~" (id 3) (at 162.56 60.96 0)
+      (effects (font (size 1.27 1.27)) hide)
+    )
+    (pin "1")
+    (pin "2")
+    (pin "3")
+    (pin "4")
+  )
+  (symbol (lib_id "Device:R_Shunt_US") (at 78.74 66.04 0) (unit 1)
+    (in_bom yes) (on_board yes) (fields_autoplaced)
+    (property "Reference" "R?" (id 0) (at 76.2 64.7699 0)
+      (effects (font (size 1.27 1.27)) (justify right))
+    )
+    (property "Value" "R_Shunt_US" (id 1) (at 76.2 67.3099 0)
+      (effects (font (size 1.27 1.27)) (justify right))
+    )
+    (property "Footprint" "" (id 2) (at 76.962 66.04 90)
+      (effects (font (size 1.27 1.27)) hide)
+    )
+    (property "Datasheet" "~" (id 3) (at 78.74 66.04 0)
+      (effects (font (size 1.27 1.27)) hide)
+    )
+    (pin "1")
+    (pin "2")
+    (pin "3")
+    (pin "4")
+  )
+  (symbol (lib_id "Connector_Generic_MountingPin:Conn_01x01_MountingPin") (at 55.88 40.64 0) (mirror y) (unit 1)
+    (in_bom yes) (on_board yes) (fields_autoplaced)
+    (property "Reference" "J?" (id 0) (at 53.34 39.7255 0)
+      (effects (font (size 1.27 1.27)) (justify left))
+    )
+    (property "Value" "Conn_01x01_MountingPin" (id 1) (at 53.34 42.2655 0)
+      (effects (font (size 1.27 1.27)) (justify left))
+    )
+    (property "Footprint" "" (id 2) (at 55.88 40.64 0)
+      (effects (font (size 1.27 1.27)) hide)
+    )
+    (property "Datasheet" "~" (id 3) (at 55.88 40.64 0)
+      (effects (font (size 1.27 1.27)) hide)
+    )
+    (pin "1")
+    (pin "MP")
+  )
+  (symbol (lib_id "bvm-library:5_Pin_Meter_With_Ext_Shunt") (at 119.38 71.12 0) (unit 1)
+    (in_bom yes) (on_board yes) (fields_autoplaced)
+    (property "Reference" "M?" (id 0) (at 124.46 55.88 0))
+    (property "Value" "5_Pin_Meter_With_Ext_Shunt" (id 1) (at 124.46 58.42 0))
+    (property "Footprint" "" (id 2) (at 119.38 71.12 0)
+      (effects (font (size 1.27 1.27)) hide)
+    )
+    (property "Datasheet" "" (id 3) (at 119.38 71.12 0)
+      (effects (font (size 1.27 1.27)) hide)
+    )
+    (pin "1")
+    (pin "2")
+    (pin "3")
+    (pin "4")
+    (pin "5")
+  )
+  (symbol (lib_id "Connector_Generic_MountingPin:Conn_01x01_MountingPin") (at 55.88 86.36 0) (mirror y) (unit 1)
+    (in_bom yes) (on_board yes)
+    (property "Reference" "J?" (id 0) (at 53.34 85.4455 0)
+      (effects (font (size 1.27 1.27)) (justify left))
+    )
+    (property "Value" "Conn_01x01_MountingPin" (id 1) (at 53.34 87.9855 0)
+      (effects (font (size 1.27 1.27)) (justify left))
+    )
+    (property "Footprint" "" (id 2) (at 55.88 86.36 0)
+      (effects (font (size 1.27 1.27)) hide)
+    )
+    (property "Datasheet" "~" (id 3) (at 55.88 86.36 0)
+      (effects (font (size 1.27 1.27)) hide)
+    )
+    (pin "1")
+    (pin "MP")
+  )
 )

Commit message: Bunch more changes
Blah blah
Parts:
- gave numbers to parts that had none: 1
Connections:
- no-connect marks 0 -> 3
Other:
- title: (none) -> Mr. Powers
Changed lines of the file:
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@@
   (paper "A4")
   (title_block
+    (title "Mr. Powers")
     (date "2022-05-20")
     (rev "0.0.0-draft")
@@
   (junction (at 179.07 68.58) (diameter 0) (color 0 0 0 0)
   )
+  (no_connect (at 55.88 101.6))
+  (no_connect (at 55.88 91.44))
+  (no_connect (at 55.88 45.72))
   (wire (pts (xy 144.78 40.64) (xy 144.78 66.04))
     (stroke (width 0) (type default) (color 0 0 0 0))
@@
     (stroke (width 0) (type default) (color 0 0 0 0))
   )
-  (wire (pts (xy 82.55 68.58) (xy 111.76 68.58))
-    (stroke (width 0) (type default) (color 0 0 0 0))
-  )
   (wire (pts (xy 179.07 68.58) (xy 182.88 68.58))
     (stroke (width 0) (type default) (color 0 0 0 0))
@@
   )
   (wire (pts (xy 152.4 68.58) (xy 157.48 68.58))
+    (stroke (width 0) (type default) (color 0 0 0 0))
+  )
+  (wire (pts (xy 82.55 68.58) (xy 111.76 68.58))
     (stroke (width 0) (type default) (color 0 0 0 0))
   )
@@
   (symbol (lib_id "Device:R_Shunt_US") (at 78.74 66.04 0) (unit 1)
     (in_bom yes) (on_board yes) (fields_autoplaced)
-    (property "Reference" "R?" (id 0) (at 76.2 64.7699 0)
+    (property "Reference" "RSHUNT_VDC_METER" (id 0) (at 76.2 64.7699 0)
       (effects (font (size 1.27 1.27)) (justify right))
     )

Commit message: Minor change across the board
I need better notes.
Parts:
- gave numbers to parts that had none: 6
- renumbered RSHUNT_VDC_METER to RSHUNT_VDC_METER1
Changed lines of the file:
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@@
   (symbol (lib_id "Connector_Generic_MountingPin:Conn_01x01_MountingPin") (at 55.88 30.48 0) (mirror y) (unit 1)
     (in_bom yes) (on_board yes) (fields_autoplaced)
-    (property "Reference" "J?" (id 0) (at 53.34 29.5655 0)
+    (property "Reference" "J7" (id 0) (at 53.34 29.5655 0)
       (effects (font (size 1.27 1.27)) (justify left))
     )
@@
   (symbol (lib_id "Connector_Generic_MountingPin:Conn_01x01_MountingPin") (at 55.88 96.52 0) (mirror y) (unit 1)
     (in_bom yes) (on_board yes) (fields_autoplaced)
-    (property "Reference" "J?" (id 0) (at 53.34 95.6055 0)
+    (property "Reference" "J10" (id 0) (at 53.34 95.6055 0)
       (effects (font (size 1.27 1.27)) (justify left))
     )
@@
   (symbol (lib_id "Switch:SW_SPST_LED") (at 162.56 68.58 0) (mirror y) (unit 1)
     (in_bom yes) (on_board yes) (fields_autoplaced)
-    (property "Reference" "SW_SYSPOWER?" (id 0) (at 163.195 59.69 0))
+    (property "Reference" "SW_SYSPOWER2" (id 0) (at 163.195 59.69 0))
     (property "Value" "SW_SPST_LED" (id 1) (at 163.195 62.23 0))
     (property "Footprint" "" (id 2) (at 162.56 60.96 0)
@@
   (symbol (lib_id "Device:R_Shunt_US") (at 78.74 66.04 0) (unit 1)
     (in_bom yes) (on_board yes) (fields_autoplaced)
-    (property "Reference" "RSHUNT_VDC_METER" (id 0) (at 76.2 64.7699 0)
+    (property "Reference" "RSHUNT_VDC_METER1" (id 0) (at 76.2 64.7699 0)
       (effects (font (size 1.27 1.27)) (justify right))
     )
@@
   (symbol (lib_id "Connector_Generic_MountingPin:Conn_01x01_MountingPin") (at 55.88 40.64 0) (mirror y) (unit 1)
     (in_bom yes) (on_board yes) (fields_autoplaced)
-    (property "Reference" "J?" (id 0) (at 53.34 39.7255 0)
+    (property "Reference" "J8" (id 0) (at 53.34 39.7255 0)
       (effects (font (size 1.27 1.27)) (justify left))
     )
@@
   (symbol (lib_id "bvm-library:5_Pin_Meter_With_Ext_Shunt") (at 119.38 71.12 0) (unit 1)
     (in_bom yes) (on_board yes) (fields_autoplaced)
-    (property "Reference" "M?" (id 0) (at 124.46 55.88 0))
+    (property "Reference" "M5" (id 0) (at 124.46 55.88 0))
     (property "Value" "5_Pin_Meter_With_Ext_Shunt" (id 1) (at 124.46 58.42 0))
     (property "Footprint" "" (id 2) (at 119.38 71.12 0)
@@
   (symbol (lib_id "Connector_Generic_MountingPin:Conn_01x01_MountingPin") (at 55.88 86.36 0) (mirror y) (unit 1)
     (in_bom yes) (on_board yes)
-    (property "Reference" "J?" (id 0) (at 53.34 85.4455 0)
+    (property "Reference" "J9" (id 0) (at 53.34 85.4455 0)
       (effects (font (size 1.27 1.27)) (justify left))
     )
